File: Flex60/Flex60.kicad_pcb (KiCad board)
At the start: 2 copper layers, 285 x 94.6 mm, 6 parts

Commit message: Layout of switches
Parts:
- added D1: BAV70, Custom_Footprints:SOT-23_Annotated, B.Cu at (126.2, -22.2)
- added D10: BAV70, Custom_Footprints:SOT-23_Annotated, B.Cu at (157.9, -26.5)
- added D11: BAV70, Custom_Footprints:SOT-23_Annotated, B.Cu at (153.5, -26.5)
- added D12: BAV70, Custom_Footprints:SOT-23_Annotated, B.Cu at (149.0, -26.5)
- added D13: BAV70, Custom_Footprints:SOT-23_Annotated, B.Cu at (144.6, -26.5)
- added D14: BAV70, Custom_Footprints:SOT-23_Annotated, B.Cu at (162.4, -22.0)
- added D15: BAV70, Custom_Footprints:SOT-23_Annotated, B.Cu at (135.7, -26.5)
- added D16: BAV70, Custom_Footprints:SOT-23_Annotated, B.Cu at (144.6, -17.4)
- added D17: BAV70, Custom_Footprints:SOT-23_Annotated, B.Cu at (149.0, -22.0)
- added D18: BAV70, Custom_Footprints:SOT-23_Annotated, B.Cu at (166.8, -17.4)
- added D19: BAV70, Custom_Footprints:SOT-23_Annotated, B.Cu at (162.4, -17.4)
- added D2: BAV70, Custom_Footprints:SOT-23_Annotated, B.Cu at (135.7, -22.0)
- added D20: BAV70, Custom_Footprints:SOT-23_Annotated, B.Cu at (157.9, -17.4)
- added D21: BAV70, Custom_Footprints:SOT-23_Annotated, B.Cu at (153.5, -17.4)
- added D22: BAV70, Custom_Footprints:SOT-23_Annotated, B.Cu at (149.0, -17.4)
- added D23: BAV70, Custom_Footprints:SOT-23_Annotated, B.Cu at (135.7, -31.1)
- added D24: BAV70, Custom_Footprints:SOT-23_Annotated, B.Cu at (140.1, -26.5)
- added D25: BAV70, Custom_Footprints:SOT-23_Annotated, B.Cu at (144.6, -22.0)
- added D26: BAV70, Custom_Footprints:SOT-23_Annotated, B.Cu at (140.1, -22.0)
- added D27: BAV70, Custom_Footprints:SOT-23_Annotated, B.Cu at (131.2, -31.1)
- added D28: BAV70, Custom_Footprints:SOT-23_Annotated, B.Cu at (157.9, -22.0)
- added D29: BAV70, Custom_Footprints:SOT-23_Annotated, B.Cu at (131.2, -26.5)
- added D3: BAV70, Custom_Footprints:SOT-23_Annotated, B.Cu at (153.5, -22.0)
- added D30: BAV70, Custom_Footprints:SOT-23_Annotated, B.Cu at (135.7, -17.4)
- added D31: BAV70, Custom_Footprints:SOT-23_Annotated, B.Cu at (131.2, -17.4)
- added D32: BAV70, Custom_Footprints:SOT-23_Annotated, B.Cu at (140.1, -17.4)
- added D33: BAV70, Custom_Footprints:SOT-23_Annotated, B.Cu at (131.2, -22.0)
- added D4: BAV70, Custom_Footprints:SOT-23_Annotated, B.Cu at (162.4, -26.5)
- added D5: BAV70, Custom_Footprints:SOT-23_Annotated, B.Cu at (157.9, -31.1)
- added D6: BAV70, Custom_Footprints:SOT-23_Annotated, B.Cu at (153.5, -31.1)
- added D7: BAV70, Custom_Footprints:SOT-23_Annotated, B.Cu at (149.0, -31.1)
- added D8: BAV70, Custom_Footprints:SOT-23_Annotated, B.Cu at (144.6, -31.1)
- added D9: BAV70, Custom_Footprints:SOT-23_Annotated, B.Cu at (140.1, -31.1)
- added K_0: KC_ESC, MX_Only:MXOnly-1U-NoLED, F.Cu at (2.52, 2.52)
- added K_013A1: KC_BSPC, MX_Only:MXOnly-1U-NoLED, F.Cu at (250.2, 2.52)
- added K_1: KC_1, MX_Only:MXOnly-1U-NoLED, F.Cu at (21.6, 2.52)
- added K_10: KC_0, MX_Only:MXOnly-1U-NoLED, F.Cu at (193.0, 2.52)
- added K_100: KC_TAB, MX_Only:MXOnly-1.5U-NoLED, F.Cu at (7.29, 21.6)
- added K_101: KC_Q, MX_Only:MXOnly-1U-NoLED, F.Cu at (31.1, 21.6)
- added K_102: KC_W, MX_Only:MXOnly-1U-NoLED, F.Cu at (50.1, 21.6)
- added K_103: KC_E, MX_Only:MXOnly-1U-NoLED, F.Cu at (69.2, 21.6)
- added K_104: KC_R, MX_Only:MXOnly-1U-NoLED, F.Cu at (88.2, 21.6)
- added K_105: KC_T, MX_Only:MXOnly-1U-NoLED, F.Cu at (107.3, 21.6)
- added K_106: KC_Y, MX_Only:MXOnly-1U-NoLED, F.Cu at (126.3, 21.6)
- added K_107: KC_U, MX_Only:MXOnly-1U-NoLED, F.Cu at (145.4, 21.6)
- added K_108: KC_I, MX_Only:MXOnly-1U-NoLED, F.Cu at (164.4, 21.6)
- added K_109: KC_O, MX_Only:MXOnly-1U-NoLED, F.Cu at (183.5, 21.6)
- added K_11: KC_MINS, MX_Only:MXOnly-1U-NoLED, F.Cu at (212.1, 2.52)
- added K_110: KC_P, MX_Only:MXOnly-1U-NoLED, F.Cu at (202.6, 21.6)
- added K_111: KC_LBRC, MX_Only:MXOnly-1U-NoLED, F.Cu at (221.6, 21.6)
- added K_112: KC_RBRC, MX_Only:MXOnly-1U-NoLED, F.Cu at (240.7, 21.6)
- added K_113: KC_BSLS, MX_Only:MXOnly-1.5U-NoLED, F.Cu at (264.5, 21.6)
- added K_12: KC_EQL, MX_Only:MXOnly-1U-NoLED, F.Cu at (231.1, 2.52)
- added K_13: KC_BSPC, MX_Only:MXOnly-2U-NoLED, F.Cu at (259.7, 2.52)
- added K_2: KC_2, MX_Only:MXOnly-1U-NoLED, F.Cu at (40.6, 2.52)
- added K_200: KC_CAPS, MX_Only:MXOnly-1.75U-NoLED, F.Cu at (9.67, 40.6)
- added K_200A1: KC_CAPS, MX_Only:MXOnly-1.25U-NoLED, F.Cu at (4.91, 40.6)
- added K_201: KC_A, MX_Only:MXOnly-1U-NoLED, F.Cu at (35.9, 40.6)
- added K_202: KC_S, MX_Only:MXOnly-1U-NoLED, F.Cu at (54.9, 40.6)
- added K_203: KC_D, MX_Only:MXOnly-1U-NoLED, F.Cu at (74.0, 40.6)
- added K_204: KC_F, MX_Only:MXOnly-1U-NoLED, F.Cu at (93.0, 40.6)
- added K_205: KC_G, MX_Only:MXOnly-1U-NoLED, F.Cu at (112.1, 40.6)
- added K_206: KC_H, MX_Only:MXOnly-1U-NoLED, F.Cu at (131.1, 40.6)
- added K_207: KC_J, MX_Only:MXOnly-1U-NoLED, F.Cu at (150.2, 40.6)
- added K_208: KC_K, MX_Only:MXOnly-1U-NoLED, F.Cu at (169.2, 40.6)
- added K_209: KC_L, MX_Only:MXOnly-1U-NoLED, F.Cu at (188.3, 40.6)
- added K_210: KC_SCLN, MX_Only:MXOnly-1U-NoLED, F.Cu at (207.3, 40.6)
- added K_211: KC_QUOT, MX_Only:MXOnly-1U-NoLED, F.Cu at (226.4, 40.6)
- added K_212: KC_ENT, MX_Only:MXOnly-2.25U-NoLED, F.Cu at (257.3, 40.6)
- added K_213: KC_DEL, MX_Only:MXOnly-1U-NoLED, F.Cu at (269.2, 2.52)
- added K_3: KC_3, MX_Only:MXOnly-1U-NoLED, F.Cu at (59.7, 2.52)
- added K_300: KC_LSFT, MX_Only:MXOnly-2.25U-NoLED, F.Cu at (14.4, 59.7)
- added K_301: KC_Z, MX_Only:MXOnly-1U-NoLED, F.Cu at (45.4, 59.7)
- added K_302: KC_X, MX_Only:MXOnly-1U-NoLED, F.Cu at (64.4, 59.7)
- added K_303: KC_C, MX_Only:MXOnly-1U-NoLED, F.Cu at (83.5, 59.7)
- added K_304: KC_V, MX_Only:MXOnly-1U-NoLED, F.Cu at (102.5, 59.7)
- added K_305: KC_B, MX_Only:MXOnly-1U-NoLED, F.Cu at (121.6, 59.7)
- added K_306: KC_N, MX_Only:MXOnly-1U-NoLED, F.Cu at (140.6, 59.7)
- added K_307: KC_M, MX_Only:MXOnly-1U-NoLED, F.Cu at (159.7, 59.7)
- added K_308: KC_COMM, MX_Only:MXOnly-1U-NoLED, F.Cu at (178.7, 59.7)
- added K_309: KC_DOT, MX_Only:MXOnly-1U-NoLED, F.Cu at (197.8, 59.7)
- added K_310: KC_SLSH, MX_Only:MXOnly-1U-NoLED, F.Cu at (216.8, 59.7)
- added K_311: KC_RSFT, MX_Only:MXOnly-2.75U-NoLED, F.Cu at (252.6, 59.7)
- added K_311A1: KC_RSFT, MX_Only:MXOnly-1.75U-NoLED, F.Cu at (243.0, 59.7)
- added K_312: KC_MO(1), MX_Only:MXOnly-1U-NoLED, F.Cu at (269.2, 59.7)
- added K_4: KC_4, MX_Only:MXOnly-1U-NoLED, F.Cu at (78.7, 2.52)
- added K_400: KC_LCTL, MX_Only:MXOnly-1.25U-NoLED, F.Cu at (4.91, 78.7)
- added K_400A1: KC_LCTL, MX_Only:MXOnly-1.5U-NoLED, F.Cu at (7.29, 78.7)
- added K_401: KC_LGUI, MX_Only:MXOnly-1.25U-NoLED, F.Cu at (28.7, 78.7)
- added K_401A1: KC_LGUI, MX_Only:MXOnly-1U-NoLED, F.Cu at (31.1, 78.7)
- added K_402: KC_LALT, MX_Only:MXOnly-1.25U-NoLED, F.Cu at (52.5, 78.7)
- added K_402A1: KC_LALT, MX_Only:MXOnly-1.5U-NoLED, F.Cu at (54.9, 78.7)
- added K_406: KC_SPC, MX_Only:MXOnly-6.25U-ReversedStabilizers-NoLED, F.Cu at (124.0, 78.7)
- added K_406A1: KC_SPC, MX_Only:MXOnly-7U-ReversedStabilizers-NoLED, F.Cu at (135.9, 78.7)
- added K_408: KC_RALT, MX_Only:MXOnly-1.25U-NoLED, F.Cu at (195.4, 78.7)
- added K_409: KC_RGUI, MX_Only:MXOnly-1.25U-NoLED, F.Cu at (219.2, 78.7)
- added K_409A1: KC_RALT, MX_Only:MXOnly-1.5U-NoLED, F.Cu at (216.8, 78.7)
- added K_410: KC_MO(1), MX_Only:MXOnly-1.25U-NoLED, F.Cu at (243.0, 78.7)
- added K_410A1: KC_MO(1), MX_Only:MXOnly-1U-NoLED, F.Cu at (240.7, 78.7)
- added K_411: KC_RCTL, MX_Only:MXOnly-1.25U-NoLED, F.Cu at (266.8, 78.7)
- added K_411A1: KC_RCTL, MX_Only:MXOnly-1.5U-NoLED, F.Cu at (264.5, 78.7)
- added K_5: KC_5, MX_Only:MXOnly-1U-NoLED, F.Cu at (97.8, 2.52)
- added K_6: KC_6, MX_Only:MXOnly-1U-NoLED, F.Cu at (116.8, 2.52)
- added K_7: KC_7, MX_Only:MXOnly-1U-NoLED, F.Cu at (135.9, 2.52)
- added K_8: KC_8, MX_Only:MXOnly-1U-NoLED, F.Cu at (154.9, 2.52)
- added K_9: KC_9, MX_Only:MXOnly-1U-NoLED, F.Cu at (174.0, 2.52)
- moved H4 23.0 mm to (121.6, 40.0)
- moved H1 22.7 mm to (-4.85, 49.5)
- moved H3 22.7 mm to (19.1, 20.9)
- moved H5 22.7 mm to (184.4, 78.2)
- moved H6 22.7 mm to (253.9, 20.9)
- moved H2 22.7 mm to (277.6, 49.5)

Commit message: Layout Diodes + add flex cuts
Parts:
- removed the D31 at (131.2, -17.4)
- moved D32 154.5 mm to (253.3, 72.6), turned to 90 degrees
- moved D29 149.6 mm to (19.2, 72.6), turned to 90 degrees
- moved D22 134.9 mm to (34.3, 53.6), turned to 90 degrees
- moved D8 133.4 mm to (19.2, 14.4), turned to 90 degrees
- moved D15 129.4 mm to (21.6, 34.5), turned to 90 degrees
- moved D27 127.4 mm to (226.4, 53.6), turned to 90 degrees
- moved D28 123.0 mm to (258.1, 49.4), turned to 90 degrees
- moved D21 117.0 mm to (260.8, 29.3), turned to 90 degrees
- moved D1 115.7 mm to (12.1, -3.53), turned to 90 degrees
- moved D31 111.0 mm to (204.9, 72.6), turned to 90 degrees
- moved D23 104.8 mm to (74.0, 53.6), turned to 90 degrees
- moved D30 98.3 mm to (96.2, 72.6), turned to 90 degrees
- moved D14 98.0 mm to (253.3, 14.4), turned to 90 degrees
- moved D7 95.7 mm to (240.7, -3.53), turned to 90 degrees
- moved D16 95.5 mm to (64.4, 34.5), turned to 90 degrees
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- renumbered D32 to D31, D33 to D32
Connections:
- D31 pad 1: Net-(D32-Pad1) -> Net-(D31-Pad1)
- D31 pad 2: Net-(D32-Pad2) -> Net-(D31-Pad2)
- D32 pad 1: Net-(D33-Pad1) -> Net-(D32-Pad1)
- D32 pad 2: Net-(D33-Pad2) -> Net-(D32-Pad2)
- K_0 pad 2: Net-(D1-Pad1) -> Net-(D1-Pad2)
- K_013A1 pad 2: Net-(D7-Pad2) -> Net-(D7-Pad1)
- K_1 pad 2: Net-(D1-Pad2) -> Net-(D1-Pad1)
- K_10 pad 2: Net-(D6-Pad1) -> Net-(D6-Pad2)
- K_100 pad 2: Net-(D8-Pad1) -> Net-(D8-Pad2)
- K_101 pad 2: Net-(D8-Pad2) -> Net-(D8-Pad1)
- K_102 pad 2: Net-(D9-Pad1) -> Net-(D9-Pad2)
- K_103 pad 2: Net-(D9-Pad2) -> Net-(D9-Pad1)
- K_104 pad 2: Net-(D10-Pad1) -> Net-(D10-Pad2)
- K_105 pad 2: Net-(D10-Pad2) -> Net-(D10-Pad1)
- K_106 pad 2: Net-(D11-Pad1) -> Net-(D11-Pad2)
- K_107 pad 2: Net-(D11-Pad2) -> Net-(D11-Pad1)
- K_108 pad 2: Net-(D12-Pad1) -> Net-(D12-Pad2)
- K_109 pad 2: Net-(D12-Pad2) -> Net-(D12-Pad1)
- K_11 pad 2: Net-(D6-Pad2) -> Net-(D6-Pad1)
- K_110 pad 2: Net-(D13-Pad1) -> Net-(D13-Pad2)
- K_111 pad 2: Net-(D13-Pad2) -> Net-(D13-Pad1)
- K_112 pad 2: Net-(D14-Pad1) -> Net-(D14-Pad2)
- K_113 pad 2: Net-(D14-Pad2) -> Net-(D14-Pad1)
- K_12 pad 2: Net-(D7-Pad1) -> Net-(D7-Pad2)
- K_13 pad 2: Net-(D7-Pad2) -> Net-(D7-Pad1)
- K_2 pad 2: Net-(D2-Pad1) -> Net-(D2-Pad2)
- K_200 pad 2: Net-(D15-Pad1) -> Net-(D15-Pad2)
- K_200A1 pad 2: Net-(D15-Pad1) -> Net-(D15-Pad2)
- K_201 pad 2: Net-(D15-Pad2) -> Net-(D15-Pad1)
- K_202 pad 2: Net-(D16-Pad1) -> Net-(D16-Pad2)
- K_203 pad 2: Net-(D16-Pad2) -> Net-(D16-Pad1)
- K_204 pad 2: Net-(D17-Pad1) -> Net-(D17-Pad2)
- K_205 pad 2: Net-(D17-Pad2) -> Net-(D17-Pad1)
- K_206 pad 2: Net-(D18-Pad1) -> Net-(D18-Pad2)
- K_207 pad 2: Net-(D18-Pad2) -> Net-(D18-Pad1)
- K_208 pad 2: Net-(D19-Pad1) -> Net-(D19-Pad2)
- K_209 pad 2: Net-(D19-Pad2) -> Net-(D19-Pad1)
- K_210 pad 2: Net-(D20-Pad1) -> Net-(D20-Pad2)
- K_211 pad 2: Net-(D20-Pad2) -> Net-(D20-Pad1)
- K_212 pad 2: Net-(D21-Pad1) -> Net-(D21-Pad2)
- K_213 pad 2: Net-(D21-Pad2) -> Net-(D21-Pad1)
- K_3 pad 2: Net-(D2-Pad2) -> Net-(D2-Pad1)
- K_300 pad 2: Net-(D22-Pad1) -> Net-(D22-Pad2)
- K_301 pad 2: Net-(D22-Pad2) -> Net-(D22-Pad1)
- K_302 pad 2: Net-(D23-Pad1) -> Net-(D23-Pad2)
- K_303 pad 2: Net-(D23-Pad2) -> Net-(D23-Pad1)
- K_304 pad 2: Net-(D24-Pad1) -> Net-(D24-Pad2)
- K_305 pad 2: Net-(D24-Pad2) -> Net-(D24-Pad1)
- K_306 pad 2: Net-(D25-Pad1) -> Net-(D25-Pad2)
- K_307 pad 2: Net-(D25-Pad2) -> Net-(D25-Pad1)
- K_308 pad 2: Net-(D26-Pad1) -> Net-(D26-Pad2)
- K_309 pad 2: Net-(D26-Pad2) -> Net-(D26-Pad1)
- K_310 pad 2: Net-(D27-Pad1) -> Net-(D27-Pad2)
- K_311 pad 2: Net-(D27-Pad2) -> Net-(D27-Pad1)
- K_311A1 pad 2: Net-(D27-Pad2) -> Net-(D27-Pad1)
- K_4 pad 2: Net-(D3-Pad1) -> Net-(D3-Pad2)
- K_400 pad 2: Net-(D29-Pad1) -> Net-(D29-Pad2)
- K_400A1 pad 2: Net-(D29-Pad1) -> Net-(D29-Pad2)
- K_401 pad 2: Net-(D29-Pad2) -> Net-(D29-Pad1)
- K_401A1 pad 2: Net-(D29-Pad2) -> Net-(D29-Pad1)
- K_402 pad 2: Net-(D30-Pad1) -> Net-(D30-Pad2)
- K_402A1 pad 2: Net-(D30-Pad1) -> Net-(D30-Pad2)
- K_406 pad 2: Net-(D31-Pad1) -> Net-(D30-Pad1)
- K_406A1 pad 2: Net-(D31-Pad1) -> Net-(D30-Pad1)
- K_408 pad 2: Net-(D32-Pad1) -> Net-(D31-Pad2)
- K_409 pad 2: Net-(D32-Pad2) -> Net-(D31-Pad1)
- K_409A1 pad 2: Net-(D32-Pad2) -> Net-(D31-Pad1)
- K_410 pad 2: Net-(D33-Pad1) -> Net-(D32-Pad2)
- K_410A1 pad 2: Net-(D33-Pad1) -> Net-(D32-Pad2)
- K_411 pad 2: Net-(D33-Pad2) -> Net-(D32-Pad1)
- K_411A1 pad 2: Net-(D33-Pad2) -> Net-(D32-Pad1)
- K_5 pad 2: Net-(D3-Pad2) -> Net-(D3-Pad1)
- K_6 pad 2: Net-(D4-Pad1) -> Net-(D4-Pad2)
- K_7 pad 2: Net-(D4-Pad2) -> Net-(D4-Pad1)
- K_8 pad 2: Net-(D5-Pad1) -> Net-(D5-Pad2)
- K_9 pad 2: Net-(D5-Pad2) -> Net-(D5-Pad1)
Other:
- outline, holes or cut-outs redrawn
