File: Flex60/Flex60.kicad_pcb (KiCad board)
At the start: 2 copper layers, 285 x 94.6 mm, 128 parts, among them SW1 RESET, U1 ATmega32U4-AU, Y1 16MHz

Commit message: Add Art + generate new gerbers
Parts:
- added G***: LOGO, FlexHoles:NODU_COW_980, B.Cu at (155.4, 79.1)
- added REF**: 12x12MakerMark, Logo:12x12MakerMark, B.Cu at (107.2, 79.6)
Other:
- board text added: "NODU"
